File: barra-monocolor/Schematics/dmx_to_pwm/dmx_to_pwm.kicad_pcb (KiCad board)
At the start: 2 copper layers, 36 parts, among them IC1 LM1085IT-12_NOPB, J4 PJ-031D, SW1 SW_SPDT, SW1 SW_SPST, SW2 SW_SPDT, SW3 SW_SPDT, U1 SN75176AP, U2 6N137, U3 6N137, U4 SN75176AP

Commit message: first pcb layout
Parts:
- removed D1: 1N4148, Diode_THT:D_DO-35_SOD27_P7.62mm_Horizontal
- removed IC1: LM1085IT-12_NOPB, Lasers:TO254P470X1028X1955-3P
- removed J4: PJ-031D, Lasers:PJ031D
- removed R11, R12, R5: 1K, Resistor_THT:R_Axial_DIN0204_L3.6mm_D1.6mm_P7.62mm_Horizontal
- removed R15: 133, Resistor_THT:R_Axial_DIN0204_L3.6mm_D1.6mm_P7.62mm_Horizontal
- removed R16, R17: 562, Resistor_THT:R_Axial_DIN0204_L3.6mm_D1.6mm_P7.62mm_Horizontal
- removed R19: 4.7K, Resistor_THT:R_Axial_DIN0204_L3.6mm_D1.6mm_P7.62mm_Horizontal
- removed the SW1 at (74.9, 69.9)
- removed the SW1 at (69.9, 80.0)
- removed SW2, SW3: SW_SPDT, Button_Switch_THT:SW_Slide-03_Wuerth-WS-SLTV_10x2.5x6.4_P2.54mm
- removed U1: SN75176AP, Package_DIP:DIP-8_W7.62mm
- added C10: 1uF, Capacitor_THT:C_Disc_D3.0mm_W2.0mm_P2.50mm, F.Cu at (276.1, 70.8)
- added C11: 1uF, Capacitor_THT:C_Disc_D3.0mm_W2.0mm_P2.50mm, F.Cu at (276.1, 74.3)
- added C12: 100nF, Capacitor_THT:C_Disc_D3.0mm_W2.0mm_P2.50mm, F.Cu at (276.1, 77.9)
- added C13: 100nF, Capacitor_THT:C_Disc_D3.0mm_W2.0mm_P2.50mm, F.Cu at (276.1, 81.5)
- added C7: 47uF - 50V, Capacitor_THT:CP_Radial_D7.5mm_P2.50mm, F.Cu at (176.5, 62.0)
- added C8: 1uF, Capacitor_THT:C_Disc_D3.0mm_W2.0mm_P2.50mm, F.Cu at (270.4, 81.5)
- added C9: 1uF, Capacitor_THT:C_Disc_D3.0mm_W2.0mm_P2.50mm, F.Cu at (276.1, 67.2)
- added D3: 1N4004, Diode_THT:D_DO-41_SOD81_P7.62mm_Horizontal, F.Cu at (194.9, 110.5)
- added D4: 1N4004, Diode_THT:D_DO-41_SOD81_P7.62mm_Horizontal, F.Cu at (194.9, 114.8)
- added D5: 1N4004, Diode_THT:D_DO-41_SOD81_P7.62mm_Horizontal, F.Cu at (194.9, 119.0)
- added D6: 1N4004, Diode_THT:D_DO-41_SOD81_P7.62mm_Horizontal, F.Cu at (194.9, 123.2)
- added J1: RJ45, Connector_RJ:RJ45_Amphenol_54602-x08_Horizontal, F.Cu at (162.4, 152.9)
- added J2: RJ45, Connector_RJ:RJ45_Amphenol_54602-x08_Horizontal, F.Cu at (145.2, 152.9)
- added J3: Conn_02x04_Top_Bottom, Connector_PinHeader_2.54mm:PinHeader_2x04_P2.54mm_Vertical, F.Cu at (152.9, 107.7)
- added J5: Conn_01x05_Socket, Connector_JST:JST_EH_B5B-EH-A_1x05_P2.50mm_Vertical, F.Cu at (138.5, 98.0)
- added L1: 100uH, Capacitor_THT:CP_Radial_D12.5mm_P7.50mm, F.Cu at (158.5, 50.0)
- added Q1: TIP41, Package_TO_SOT_THT:TO-220-3_Vertical, F.Cu at (162.9, 73.8)
- added Q2: TIP41, Package_TO_SOT_THT:TO-220-3_Vertical, F.Cu at (162.9, 79.7)
- added Q3: TIP41, Package_TO_SOT_THT:TO-220-3_Vertical, F.Cu at (162.9, 85.7)
- added Q5: TIP41, Package_TO_SOT_THT:TO-220-3_Vertical, F.Cu at (162.9, 91.7)
- added RV1: 20, Potentiometer_THT:Potentiometer_Bourns_3296Z_Horizontal, F.Cu at (228.0, 83.5)
- added RV2: 20, Potentiometer_THT:Potentiometer_Bourns_3296Z_Horizontal, F.Cu at (228.0, 90.0)
- added RV3: 20, Potentiometer_THT:Potentiometer_Bourns_3296Z_Horizontal, F.Cu at (252.7, 109.0)
- added RV4: 20, Potentiometer_THT:Potentiometer_Bourns_3296Z_Horizontal, F.Cu at (252.2, 118.0)
- added SW1: SW_DIP_x08, Package_DIP:DIP-16_W7.62mm_LongPads, F.Cu at (233.0, 83.6)
- added U5: LM337_TO220, Package_TO_SOT_THT:TO-220-3_Vertical, F.Cu at (162.9, 109.5)
- added U6: LM337_TO220, Package_TO_SOT_THT:TO-220-3_Vertical, F.Cu at (162.9, 115.5)
- added U8: SN75176AP, Package_DIP:DIP-8_W7.62mm_Socket_LongPads, F.Cu at (220.4, 109.5)
- added U9: H11L1, Package_DIP:DIP-6_W7.62mm_LongPads, F.Cu at (157.2, 131.5)
- C1: value 100nF -> 47uF - 50V; footprint Capacitor_THT:C_Disc_D3.0mm_W2.0mm_P2.50mm -> Capacitor_THT:CP_Radial_D7.5mm_P2.50mm
- C3: value 10uF -> 100nF; footprint Capacitor_THT:CP_Radial_Tantal_D5.5mm_P2.50mm -> Capacitor_THT:C_Disc_D3.0mm_W2.0mm_P2.50mm
- C4: value 330nF -> 100nF; footprint Capacitor_THT:CP_Radial_Tantal_D5.5mm_P2.50mm -> Capacitor_THT:C_Disc_D3.0mm_W2.0mm_P2.50mm
- D2: value 1N4148 -> 1N5822; footprint Diode_THT:D_DO-35_SOD27_P7.62mm_Horizontal -> Diode_THT:D_DO-201AD_P15.24mm_Horizontal
- R1, R2, R3, R4: footprint Resistor_THT:R_Axial_DIN0204_L3.6mm_D1.6mm_P7.62mm_Horizontal -> Resistor_THT:R_Axial_DIN0414_L11.9mm_D4.5mm_P7.62mm_Vertical
- R10: value 1K -> 470; footprint Resistor_THT:R_Axial_DIN0204_L3.6mm_D1.6mm_P7.62mm_Horizontal -> Resistor_THT:R_Axial_DIN0414_L11.9mm_D4.5mm_P7.62mm_Vertical
- R13: value 470 -> 10K; footprint Resistor_THT:R_Axial_DIN0204_L3.6mm_D1.6mm_P7.62mm_Horizontal -> Resistor_THT:R_Axial_DIN0414_L11.9mm_D4.5mm_P7.62mm_Vertical
- R14: value 4.7K -> 470; footprint Resistor_THT:R_Axial_DIN0204_L3.6mm_D1.6mm_P7.62mm_Horizontal -> Resistor_THT:R_Axial_DIN0414_L11.9mm_D4.5mm_P7.62mm_Vertical
- R6, R7, R8, R9: value 1K -> 2.7; footprint Resistor_THT:R_Axial_DIN0204_L3.6mm_D1.6mm_P7.62mm_Horizontal -> Resistor_THT:R_Axial_DIN0411_L9.9mm_D3.6mm_P12.70mm_Horizontal
- U2: value 6N137 -> LM2596T-5; footprint Package_DIP:DIP-8_W7.62mm -> Package_TO_SOT_THT:TO-220-5_P3.4x3.7mm_StaggerOdd_Lead3.8mm_Vertical
- U3: value 6N137 -> LM337_TO220; footprint Package_DIP:DIP-8_W7.62mm -> Package_TO_SOT_THT:TO-220-3_Vertical
- U4: value SN75176AP -> LM337_TO220; footprint Package_DIP:DIP-8_W7.62mm -> Package_TO_SOT_THT:TO-220-3_Vertical
- moved C4 237.4 mm to (270.4, 74.3)
- moved C3 217.1 mm to (270.4, 70.8)
- moved R7 191.4 mm to (220.3, 68.7), turned to 0 degrees
- moved R9 189.6 mm to (220.3, 79.0), turned to 0 degrees
- moved R8 189.2 mm to (220.3, 73.8), turned to 0 degrees
- moved R6 188.3 mm to (220.3, 63.5), turned to 0 degrees
- moved C5 185.6 mm to (270.4, 77.9)
- moved C2 184.7 mm to (270.4, 67.2)
- moved R4 166.8 mm to (194.9, 79.9), turned to 0 degrees
- moved R3 166.0 mm to (194.9, 73.8), turned to 0 degrees
- moved R10 165.4 mm to (194.9, 86.0), turned to 0 degrees
- moved R2 165.3 mm to (194.9, 67.8), turned to 0 degrees
- moved R1 164.6 mm to (194.9, 61.8), turned to 0 degrees
- moved R14 145.3 mm to (194.9, 98.0)
- moved U3 130.5 mm to (162.9, 97.6)
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Connections:
- A1 pad 10: DATA6 -> unconnected-(A1-D7-Pad10)
- A1 pad 11: DATA7 -> unconnected-(A1-D8-Pad11)
- A1 pad 12: DATA8 -> LASER4
- A1 pad 13: DATA9 -> unconnected-(A1-D10-Pad13)
- A1 pad 14: DATA10 -> unconnected-(A1-D11-Pad14)
- A1 pad 15: DATA11 -> unconnected-(A1-D12-Pad15)
- A1 pad 16: DATA12 -> unconnected-(A1-D13-Pad16)
- A1 pad 19: unconnected-(A1-A0-Pad19) -> SW1
- A1 pad 20: unconnected-(A1-A1-Pad20) -> SW2
- A1 pad 21: unconnected-(A1-A2-Pad21) -> SW3
- A1 pad 22: unconnected-(A1-A3-Pad22) -> SW4
- A1 pad 23: unconnected-(A1-A4-Pad23) -> SW5
- A1 pad 24: unconnected-(A1-A5-Pad24) -> SW6
- A1 pad 25: unconnected-(A1-A6-Pad25) -> SW7
- A1 pad 26: unconnected-(A1-A7-Pad26) -> SW8
- A1 pad 27: unconnected-(A1-+5V-Pad27) -> 5V
- A1 pad 29: DRV1- -> GND
- A1 pad 30: VIN -> unconnected-(A1-VIN-Pad30)
- A1 pad 4: DRV1- -> GND
- A1 pad 5: DATA1 -> unconnected-(A1-D2-Pad5)
- A1 pad 6: DATA2 -> LASER1
- A1 pad 7: DATA3 -> unconnected-(A1-D4-Pad7)
- A1 pad 8: DATA4 -> LASER2
- A1 pad 9: DATA5 -> LASER3
- C1 pad 1: VCC -> VIN
- C1 pad 2: DRV1- -> GND
- C2 pad 1: VCC -> 5V
- C2 pad 2: DRV1- -> Net-(J3-Pin_5)
- C3 pad 1: TO_POE_UNREG -> 5V
- C3 pad 2: DRV1- -> Net-(J3-Pin_6)
- C4 pad 1: UNREGULATED_IN -> 5V
- C4 pad 2: DRV1- -> Net-(J3-Pin_7)
- C5 pad 1: Net-(D2-A) -> 5V
- C5 pad 2: DRV1- -> Net-(J3-Pin_8)
- D2 pad 1: VIN -> GND
- R1 pad 1: DATA2 -> Net-(Q5-B)
- R1 pad 2: DRV2+ -> LASER1
- R10 pad 1: DATA10 -> Net-(R10-Pad1)
- R10 pad 2: DRV10+ -> Net-(U8-R)
- R13 pad 1: Net-(U1-R) -> GND
- R13 pad 2: Net-(U2-A) -> Net-(U8-DE)
- R14 pad 1: VCC -> 5V
- R2 pad 1: DATA3 -> Net-(Q1-B)
- R2 pad 2: DRV3+ -> LASER2
- R3 pad 1: DATA4 -> Net-(Q2-B)
- R3 pad 2: DRV4+ -> LASER3
- R4 pad 1: DATA5 -> Net-(Q3-B)
- R4 pad 2: DRV5+ -> LASER4
- R6 pad 1: DATA7 -> Net-(R6-Pad1)
- R6 pad 2: DRV7+ -> Net-(U5-VO)
- R7 pad 1: DATA1 -> Net-(R7-Pad1)
- R7 pad 2: DRV1+ -> Net-(U6-VO)
- R8 pad 1: DATA8 -> Net-(R8-Pad1)
- R8 pad 2: DRV8+ -> Net-(U4-VO)
- R9 pad 1: DATA9 -> Net-(R9-Pad1)
- R9 pad 2: DRV9+ -> Net-(U3-VO)
- U2 pad 1: unconnected-(U2-NC-Pad1) -> VIN
- U2 pad 2: Net-(U2-A) -> Net-(D2-A)
- U2 pad 3: DRV1- -> GND
- U2 pad 4: unconnected-(U2-NC-Pad4) -> 5V
- U2 pad 5: DRV1- -> GND
- U3 pad 1: unconnected-(U3-NC-Pad1) -> Net-(D6-A)
- U3 pad 2: Net-(U2-A) -> Net-(J3-Pin_8)
- U3 pad 3: DRV1- -> Net-(U3-VO)
- U4 pad 1: unconnected-(U4-R-Pad1) -> Net-(D5-A)
- U4 pad 2: VCC -> Net-(J3-Pin_7)
- U4 pad 3: VCC -> Net-(U4-VO)
Other:
- board outline added: 46 x 128 mm

Commit message: added board
Parts:
- R14: value 470 -> 1K
- moved RV4 199.0 mm to (72.4, 32.5), turned to -90 degrees
- moved C12 199.0 mm to (99.1, 168.9)
- moved C5 195.8 mm to (74.9, 66.1), turned to -90 degrees
- moved C4 190.6 mm to (80.0, 66.1), turned to -90 degrees
- moved RV3 190.0 mm to (78.7, 32.5), turned to -90 degrees
- moved C3 185.4 mm to (85.1, 66.1), turned to -90 degrees
- moved C2 180.2 mm to (90.2, 66.1), turned to -90 degrees
- moved C11 179.1 mm to (104.1, 24.1), turned to 180 degrees
- moved C10 176.3 mm to (104.1, 31.8), turned to 180 degrees
- moved C13 176.3 mm to (105.4, 125.7), turned to 180 degrees
- moved C9 174.2 mm to (104.1, 39.4), turned to 180 degrees
- moved C8 169.8 mm to (104.1, 47.0), turned to 180 degrees
- moved SW1 163.7 mm to (77.5, 134.6), turned to 90 degrees
- moved R9 154.7 mm to (71.1, 38.1), turned to -90 degrees
- moved RV2 154.0 mm to (85.1, 32.5), turned to -90 degrees
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Connections:
- net Net-(J3-Pin_3) renamed L3-SOC-IN
- net Net-(J3-Pin_6) renamed L2-SOC-OUT
- C1 pad 1: VIN -> VCC
- C2 pad 2: Net-(J3-Pin_5) -> L1-SOC-OUT
- C4 pad 2: Net-(J3-Pin_7) -> L3-SOC-OUT
- C5 pad 2: Net-(J3-Pin_8) -> L4-SOC-OUT
- D2 pad 1: GND -> Net-(D2-K)
- D2 pad 2: Net-(D2-A) -> GND
- J3 pad 1: Net-(J3-Pin_1) -> L4-SOC-IN
- J3 pad 2: Net-(J3-Pin_2) -> L4-SOC-OUT
- J3 pad 4: Net-(J3-Pin_4) -> L3-SOC-OUT
- J3 pad 5: Net-(J3-Pin_5) -> L2-SOC-IN
- J3 pad 7: Net-(J3-Pin_7) -> L1-SOC-IN
- J3 pad 8: Net-(J3-Pin_8) -> L1-SOC-OUT
- L1 pad 1: Net-(D2-A) -> Net-(D2-K)
- Q1 pad 2: Net-(J3-Pin_2) -> L2-SOC-IN
- Q3 pad 2: Net-(J3-Pin_4) -> L4-SOC-IN
- Q5 pad 2: Net-(J3-Pin_1) -> L1-SOC-IN
- U2 pad 1: VIN -> VCC
- U2 pad 2: Net-(D2-A) -> Net-(D2-K)
- U3 pad 2: Net-(J3-Pin_8) -> L4-SOC-OUT
- U4 pad 2: Net-(J3-Pin_7) -> L3-SOC-OUT
- U5 pad 2: Net-(J3-Pin_5) -> L1-SOC-OUT
Routing:
- net GND: track 0.00 -> 241.7 mm
- net 5V: track 0.00 -> 224.1 mm
- net Net-(D6-A): track 0.00 -> 80.6 mm
- net Net-(D5-A): track 0.00 -> 76.8 mm
- net Net-(D4-A): track 0.00 -> 73.5 mm
- net Net-(D3-A): track 0.00 -> 62.6 mm
- net VCC: track 0.00 -> 49.6 mm
- net Net-(A1-D0/RX): track 0.00 -> 41.3 mm
- net DATA+: track 0.00 -> 38.7 mm
- net Net-(D2-K): track 0.00 -> 32.3 mm
- net DATA-: track 0.00 -> 31.1 mm
- net L4-SOC-OUT: track 0.00 -> 21.2 mm
- net L1-SOC-OUT: track 0.00 -> 20.2 mm
- net L3-SOC-OUT: track 0.00 -> 19.7 mm
- net L2-SOC-OUT: track 0.00 -> 18.6 mm
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Other:
- board size 46 x 128 mm -> 46 x 162.3 mm
